Commit message: rosflight_sil added; clean-up and RC integration needed

File: rosflight_sim/xacro/multirotor.urdf.xacro (robot description, xacro)
@@ -43,4 +43,49 @@
     </collision>
   </link>
+  <!-- define and attach camera to base link -->
+        <link name="${namespace}/camera_link">
+          <inertial>
+            <mass value="0.000001"/>
+            <inertia ixx="0.000001" ixy="0.000001" ixz="0.000001" iyy="0.000001" iyz="0.000001" izz="0.000001"/>
+            <origin xyz="0 0 0"/>
+          </inertial>
+        </link>
+        <joint name="base_to_camera" type="fixed">
+          <origin xyz="0.5 0 0" rpy="0 0 0"/>
+          <parent link="${namespace}/base_link"/>
+          <child link="${namespace}/camera_link"/>
+        </joint>
+        <gazebo reference="${namespace}/camera_link">
+          <sensor type="camera" name="${namespace}/camera">
+            <always_on>true</always_on>
+            <update_rate>30</update_rate>
+            <camera>
+              <horizontal_fov>0.7274</horizontal_fov>
+              <image>
+                <format>R8G8B8</format>
+                <width>640</width>
+                <height>480</height>
+              </image>
+              <clip>
+                <near>0.01</near>
+                <far>1000</far>
+              </clip>
+            </camera>
+            <plugin name="camera_controller" filename="libgazebo_ros_camera.so">
+              <alwaysOn>true</alwaysOn>
+              <updateRate>0.0</updateRate>
+              <cameraName>camera</cameraName>
+              <imageTopicName>rgb</imageTopicName>
+              <cameraInfoTopicName>camera_info</cameraInfoTopicName>
+              <frameName>camera_link</frameName>
+              <hackBaseline>0.07</hackBaseline>
+              <distortionK1>0.0</distortionK1>
+              <distortionK2>0.0</distortionK2>
+              <distortionK3>0.0</distortionK3>
+              <distortionT1>0.0</distortionT1>
+              <distortionT2>0.0</distortionT2>
+            </plugin>
+          </sensor>
+        </gazebo>
   <gazebo reference="${namespace}/base_link">
     <material>Gazebo/${color}</material>
